File: hardware/battery_can_monitor/battery_can_monitor.kicad_pcb (KiCad board)
At the start: 2 copper layers, 82 x 102 mm, 71 parts, among them J1 sense3, J10 int, J11 GPIO, J12 GPIO, J13 power, J14 CAN_PWR, J15 CANGND, J2 sense1, J3 Conn_01x05_Male, J4 RJ45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

Commit message: Fix name of connectors (sense1/sense2 swapped)
Parts:
- J2: value sense1 -> sense2
- J6: value sense2 -> sense1
Connections:
- U1 pad 4: (no net) -> Net-(U1-Pad4)
- U1 pad 5: (no net) -> Net-(U1-Pad5)
- U1 pad 7: (no net) -> Net-(U1-Pad7)
